File: SOIC-8-N_to_DIP-8.sch (EAGLE design)
At the start: 3 parts, among them J1 CONNECTOR_4-0.100_VERTICAL, J2 CONNECTOR_4_PINS_5-8, U1 DS9638CM

Commit message: Updated last saved time of SOIC-8-N schematic.
Other:
- note added: "SOIC-8-N SOIC127P62X175-8N TI DS9638CM"
- note removed: "TI DS9638CM SOIC-8 SOIC127P62X175-8N"
Changed lines of the file:
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@@
 <sheet>
 <plain>
-<text x="148.59" y="24.13" size="2.54" layer="88">TI DS9638CM
-SOIC-8
-SOIC127P62X175-8N</text>
+<text x="148.59" y="24.13" size="2.54" layer="88">SOIC-8-N
+SOIC127P62X175-8N
+TI DS9638CM</text>
 </plain>
 <instances>
