File: QFN-16_with_EP_to_DIP-17.sch (EAGLE design)
At the start: 3 parts, among them J1 CONNECTOR_8, J2 CONNECTOR_9, U1 QFN-16_WITH_EP-QFN-16_EP

Commit message: Fixed text on the bottom of TQFP-32 breakout.
Other:
- note added: "QFN-16 DS28E17 QFN65P400X400X80-17N"
Changed lines of the file:
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@@
 <sheet>
 <plain>
+<text x="149.86" y="24.13" size="2.54" layer="89">QFN-16
+DS28E17
+QFN65P400X400X80-17N</text>
 </plain>
 <instances>
@@
 </schematic>
 </drawing>
+<compatibility>
+<note version="6.3" minversion="6.2.2" severity="warning">
+Since Version 6.2.2 text objects can contain more than one line,
+which will not be processed correctly with this version.
+</note>
+</compatibility>
 </eagle>
