File: TQFP-32_to_DIP-32.brd (EAGLE design)
At the start: 40.6 x 17.8 mm, 3 parts, among them J1 CONNECTOR_16, J2 CONNECTOR_16-NO_SQUARE, U1 IC-GENERIC-TQFP-32

Commit message: Fixed text on the bottom of TQFP-32 breakout.
Other:
- board text removed: "QFN-16"
Changed lines of the file:
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@@
 <layer number="14" name="Route14" color="1" fill="6" visible="no" active="no"/>
 <layer number="15" name="Route15" color="4" fill="6" visible="no" active="no"/>
-<layer number="16" name="Bottom" color="1" fill="1" visible="yes" active="yes"/>
+<layer number="16" name="Bottom" color="1" fill="1" visible="no" active="yes"/>
 <layer number="17" name="Pads" color="2" fill="1" visible="yes" active="yes"/>
 <layer number="18" name="Vias" color="2" fill="1" visible="yes" active="yes"/>
-<layer number="19" name="Unrouted" color="6" fill="1" visible="yes" active="yes"/>
+<layer number="19" name="Unrouted" color="6" fill="1" visible="no" active="yes"/>
 <layer number="20" name="Dimension" color="24" fill="1" visible="yes" active="yes"/>
 <layer number="21" name="tPlace" color="7" fill="1" visible="yes" active="yes"/>
@@
 <wire x1="39.37" y1="0" x2="0" y2="0" width="0" layer="20"/>
 <text x="1.27" y="3.81" size="1.778" layer="21" font="vector" rot="R90" align="center">1</text>
-<text x="11.176" y="5.969" size="1.778" layer="22" font="vector" rot="MR0">SnapEDA</text>
-<text x="10.541" y="2.286" size="1.778" layer="22" font="vector" rot="MR0">QFN-16</text>
 <text x="39.37" y="4.445" size="1.778" layer="21" font="vector" rot="R90" align="center">16</text>
 <text x="3.81" y="3.81" size="1.778" layer="21" font="vector" rot="R90" align="center">2</text>
@@
 <text x="6.985" y="8.89" size="1.778" layer="21" font="vector" align="center">SnapEDA</text>
 <text x="33.02" y="8.89" size="1.778" layer="21" font="vector" align="center">TQFP-32</text>
+<text x="33.02" y="8.89" size="1.778" layer="22" font="vector" rot="MR0" align="center">SnapEDA</text>
+<text x="6.985" y="8.89" size="1.778" layer="22" font="vector" rot="MR0" align="center">TQFP-32</text>
 </plain>
 <attributes>
