File: TQFP-100_to_breadboard-100.sch (EAGLE design)
At the start: 5 parts, among them J1 CONNECTOR_25, J2 CONNECTOR_25_NO_SQUARE, J3 CONNECTOR_25_NO_SQUARE, J4 CONNECTOR_25_NO_SQUARE, U1 IC-GENERIC-100-TQFP

Commit message: added TQFP-100 schematic PDF.  Added example IC P/N ATMEGA2560V-8AU to text on schematic.
Other:
- note added: "TQFP-100 DSPIC33FJ64GP310-I ATMEGA2560V-8AU"
- note removed: "TQFP-100 DSPIC33FJ64GP310-I"
Changed lines of the file:
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@@
 <text x="149.86" y="24.13" size="2.54" layer="89">TQFP-100
 DSPIC33FJ64GP310-I
-</text>
+ATMEGA2560V-8AU</text>
 </plain>
 <instances>
